File: Muscle Display.sch (EAGLE design)
At the start: 29 parts, among them IC1 MAX3232CPE, IC2 MEGA164P/324P/644P-PU, IC3 7805TV, IC5 LD117AS50TR, SW1 MINI_SWITCH

Commit message: Detatiled images for readme
Other:
- note added: "Muscle LED Display"
- note removed: "*Calulate trace size with trace width calculator External Layers in Air 10 mils are the minimum trace width 24 mil : nice "typical" width Bigger the better Spaces between traces: 8-10 Auto-route not recommended Up-size via size You can change pins if needed"
- note removed: "Final Project: CPHE-380"
- note removed: "Jonathan Batchelder"
- note removed: "Power for LED display Connect GND of Muscle sensor to LED"
- note removed: "Same Ground as battery"
